File: Peripherals.kicad_sch (KiCad schematic)
At the start: 7 parts, among them J1 Conn_01x05_Pin, J2 Conn_01x03_Pin, J3 Conn_01x03_Pin, J4 Conn_01x03_Pin, J5 Conn_01x03_Pin, J6 Conn_01x04_Pin, J7 Conn_01x04_Pin

Commit message: Updated PCB Design and footprints
Parts:
- J2, J4: footprint Connector_PinHeader_1.27mm:PinHeader_1x03_P1.27mm_Vertical -> Connector_Wire:SolderWire-2sqmm_1x03_P7.8mm_D2mm_OD3.9mm
- J3, J5: footprint Connector_PinHeader_1.27mm:PinHeader_1x03_P1.27mm_Vertical -> Connector_PinHeader_2.54mm:PinHeader_1x03_P2.54mm_Vertical
Connections:
- net +5V: now also J3.2 (Pin_2), J5.2 (Pin_2); no longer J3.3 (Pin_3), J5.3 (Pin_3)
- net GND: now also J3.3 (Pin_3); no longer J3.1 (Pin_1)
- net W1_PWM: now also J3.1 (Pin_1); no longer J3.2 (Pin_2)
- net W2_PWM: now also J5.3 (Pin_3); no longer J5.2 (Pin_2)
