File: pm_ciruit.kicad_sch (KiCad schematic)
At the start: 19 parts, among them U1 TPS54202DDC, U2 TPS7A20xxxDQN

Commit message: Updated PCB Design and footprints
Parts:
- J_BAT1: footprint Connector_PinHeader_1.27mm:PinHeader_1x02_P1.27mm_Horizontal -> Connector_Wire:SolderWire-1.5sqmm_1x02_P6mm_D1.7mm_OD3mm
- U2: footprint Package_SON:Texas_X2SON-4_1x1mm_P0.65mm -> Package_TO_SOT_SMD:SOT-23-5
Changed lines of the file:
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@@
 			)
 		)
-		(property "Footprint" "Package_SON:Texas_X2SON-4_1x1mm_P0.65mm"
+		(property "Footprint" "Package_TO_SOT_SMD:SOT-23-5"
 			(at 246.38 90.17 0)
 			(hide yes)
@@
 			)
 		)
-		(property "Footprint" "Connector_PinHeader_1.27mm:PinHeader_1x02_P1.27mm_Horizontal"
+		(property "Footprint" "Connector_Wire:SolderWire-1.5sqmm_1x02_P6mm_D1.7mm_OD3mm"
 			(at 49.53 81.28 0)
 			(hide yes)
